Commit message: adding in joint to urdf model

File: Software/offline/simulations/catkin_ws/src/RoboclubBuggy_description/urdf/RoboclubBuggy.urdf (robot description, URDF)
Before this commit: robot buggy, 1 links, 0 joints
Links:
- added link left_wheel, mass 2; collision cylinder length=0.2 radius=0.1; visual cylinder length=0.2 radius=0.1
- link chassis: mass 1 -> 2
Joints:
- added joint left_wheel_hinge: type revolute, parent chassis, child left_wheel, origin xyz=0.2 0.01 0 rpy=0 0 0, axis 0 0 1, limit lower=0.0 upper=0.548 effort=1000.0 velocity=0.5
